Commit message: Update smr200.urdf

File: urdf/smr200.urdf (robot description, URDF)
Before this commit: robot smr200, 32 links, 31 joints
Joints:
- removed joint wheel_right_
- added joint wheel_right_joint: type continuous, parent swing_arm_right_link, child wheel_right_link, origin xyz=-0.1575 -0.054 0.037 rpy=0 0 0, axis 0 0 1, limit effort=100 velocity=50

Commit message: Update smr200.urdf

File: urdf/smr200.urdf (robot description, URDF)
Before this commit: robot smr200, 32 links, 31 joints
Joints:
- joint wheel_right_joint: axis 0 0 1 -> 0 0 -1

Commit message: Add files via upload

File: urdf/smr200.urdf (robot description, URDF)
Before this commit: robot smr200, 32 links, 31 joints
Links:
- added link depthcam_front_left_view_link, mass 0.001
Joints:
- added joint depthcam_front_left_view_joint: type fixed, parent depthcam_front_left_link, child depthcam_front_left_view_link, origin xyz=0.0 0.0 0.0 rpy=-1.5708 0.0 -1.5708

Commit message: Add files via upload

File: urdf/smr200.urdf (robot description, URDF)
Before this commit: robot smr200, 33 links, 32 joints
Links:
- added link depthcam_front_right_view_link, mass 0.001
- added link lidar_merged_link
Joints:
- added joint base_link_to_lidar_merged_link: type fixed, parent base_link, child lidar_merged_link, origin xyz=0.0 0.0 -0.14228 rpy=0 0 0
- added joint depthcam_front_right_view_joint: type fixed, parent depthcam_front_right_link, child depthcam_front_right_view_link, origin xyz=0.0 0.0 0.0 rpy=-1.5708 0.0 -1.5708

Commit message: Add files via upload

File: urdf/smr200.urdf (robot description, URDF)
Before this commit: robot smr200, 35 links, 34 joints
Links:
- removed link depthcam_front_left_view_link
- removed link depthcam_front_right_view_link
- removed link lidar_merged_link
Joints:
- removed joint base_link_to_lidar_merged_link
- removed joint depthcam_front_left_view_joint
- removed joint depthcam_front_right_view_joint
- removed joint wheel_right_joint
- added joint wheel_right_: type continuous, parent swing_arm_right_link, child wheel_right_link, origin xyz=-0.1575 -0.054 0.037 rpy=0 0 0, axis 0 0 1, limit effort=100 velocity=50

Commit message: Add files via upload

File: urdf/smr200.urdf (robot description, URDF)
Before this commit: robot smr200, 32 links, 31 joints
Links:
- added link depthcam_front_left_view_link, mass 0.001
- added link depthcam_front_right_view_link, mass 0.001
- added link lidar_merged_link
Joints:
- removed joint wheel_right_
- added joint base_link_to_lidar_merged_link: type fixed, parent base_link, child lidar_merged_link, origin xyz=0.0 0.0 -0.14228 rpy=0 0 0
- added joint depthcam_front_left_view_joint: type fixed, parent depthcam_front_left_link, child depthcam_front_left_view_link, origin xyz=0.0 0.0 0.0 rpy=-1.5708 0.0 -1.5708
- added joint depthcam_front_right_view_joint: type fixed, parent depthcam_front_right_link, child depthcam_front_right_view_link, origin xyz=0.0 0.0 0.0 rpy=-1.5708 0.0 -1.5708
- added joint wheel_right_joint: type continuous, parent swing_arm_right_link, child wheel_right_link, origin xyz=-0.1575 -0.054 0.037 rpy=0 0 0, axis 0 0 -1, limit effort=100 velocity=50
